File: PCB Layout Files Kicad/Smartarter - 40/Smartarter.sch (KiCad schematic (older format))
At the start: 41 parts, among them J1 Screw_Terminal_01x03, J2 Screw_Terminal_01x03, K1 onRelay, K2 offRelay, Q1 BC547, Q2 BC547, Q3 BC547, SW1 SW_Push, U1 74164, U2 KCSA02-107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

Commit message: inductor and full wave rectifier implemented in both schematic and layout
Parts:
- removed J1, J2: Screw_Terminal_01x03, Connector_Phoenix:TerminalBlock_Phoenix_MKDS-3-3-5.08_1x03_P5.08mm_Horizontal, symbol Connector:Screw_Terminal_01x03
- removed R15: R, Resistor_THT:R_Axial_DIN0207_L6.3mm_D2.5mm_P10.16mm_Horizontal, symbol Device:R
- added C2: C_Small, Capacitor_THT:C_Disc_D3.4mm_W2.1mm_P2.50mm, symbol Device:C_Small
- added D6, D7, D8, D9: DIODE, Diode_THT:D_A-405_P2.54mm_Vertical_AnodeUp, symbol pspice:DIODE
- added J1, J2: Screw_Terminal_01x02, TerminalBlock:TerminalBlock_bornier-2_P5.08mm, symbol Connector:Screw_Terminal_01x02
- added L1: INDUCTOR, Inductor_THT:L_Axial_L9.5mm_D4.0mm_P12.70mm_Horizontal_Fastron_SMCC, symbol pspice:INDUCTOR
Connections:
- wire segments 171 -> 190
Other:
- note removed: "offRelay"
- note removed: "onRelay"

Commit message: chaar bilang chhota kar diya
Connections:
- wire segments 190 -> 193
Changed lines of the file:
@@
 Wire Wire Line
 	9850 3300 9450 3300
-Wire Wire Line
-	9450 3200 9700 3200
 Text Notes 8600 4100 1    50   ~ 0
 5V
@@
 Wire Wire Line
 	8750 3900 8750 4550
-Connection ~ 9700 3200
-Wire Wire Line
-	9700 3200 9850 3200
 Connection ~ 10150 3050
 Wire Wire Line
-	9550 3050 9550 3800
+	9550 3050 9550 3200
 Wire Wire Line
 	9550 3800 8450 3800
@@
 	0    1    1    0
 $EndComp
-Wire Wire Line
-	7200 8750 8150 8750
 $Comp
 L Connector:Screw_Terminal_01x02 J2
@@
 $EndComp
 Wire Wire Line
-	9450 3050 9550 3050
-Connection ~ 9550 3050
-Wire Wire Line
 	9100 3400 9100 2850
 Wire Wire Line
@@
 	6650 6050 6650 5950
 Wire Wire Line
+	7200 8750 8150 8750
+Wire Wire Line
+	9700 3200 9850 3200
+Wire Wire Line
+	9450 3050 9450 3100
+Wire Wire Line
+	9450 3100 9700 3100
+Wire Wire Line
+	9700 3100 9700 3200
+Connection ~ 9700 3200
+Wire Wire Line
+	9450 3200 9550 3200
+Wire Wire Line
+	7300 8650 8150 8650
+Wire Wire Line
+	7400 8550 8150 8550
+Wire Wire Line
+	7500 8450 8150 8450
+Wire Wire Line
+	7200 8350 8150 8350
+Wire Wire Line
+	7300 8250 8150 8250
+Wire Wire Line
+	7500 8050 8150 8050
+Wire Wire Line
 	7400 8150 8150 8150
-Wire Wire Line
-	7500 8050 8150 8050
-Wire Wire Line
-	7300 8250 8150 8250
-Wire Wire Line
-	7200 8350 8150 8350
-Wire Wire Line
-	7500 8450 8150 8450
-Wire Wire Line
-	7400 8550 8150 8550
-Wire Wire Line
-	7300 8650 8150 8650
 Wire Bus Line
-	8000 7900 8000 8950
+	10750 7950 10750 8950
+Wire Bus Line
+	9750 7750 9750 8950
 Wire Bus Line
 	8850 7750 8850 8950
 Wire Bus Line
-	9750 7750 9750 8950
-Wire Bus Line
-	10750 7950 10750 8950
+	8000 7900 8000 8950
+Connection ~ 9550 3200
+Wire Wire Line
+	9550 3200 9550 3800
 $EndSCHEMATC
