File: PCB Layout Files Kicad/Smartarter - 40/Smartarter.sch (KiCad schematic (older format))
At the start: 46 parts, among them J1 Screw_Terminal_01x02, J2 Screw_Terminal_01x02, K1 onRelay, K2 offRelay, Q1 BC547, Q2 BC547, Q3 BC547, SW1 SW_Push, U1 74164, U2 KCSA02-107, U3 slideSwitch, U4 7414, U5 KCSA02-107, U6 KCSA02-107, U7 KCSA02-107

Commit message: all tracks set in 40; double check the connections and HOLA ;)
Parts:
- removed U3: slideSwitch, Button_Switch_THT:SW_6-Pin-Switch_Self_Lock_DPDT_Latching, symbol Analog_Switch:DG308AxJ
- added SW2: SW_DPDT_x2, Button_Switch_THT:SW_6-Pin-Switch_Self_Lock_DPDT_Latching, symbol Switch:SW_DPDT_x2
- added digit2, digit2.1, digit3, digit3.1: HEADER-1x01, Connector_Wire:SolderWirePad_1x01_Drill0.8mm, symbol connectors:HEADER-1x01
- renumbered RV1 to POT1, U4 to U7414, U1 to U74164, D1 to green1, K2 to offRelay1, K1 to onRelay1, D2 to red1, D3 to yellow1
Connections:
- net labels added: CLK, D1, D4, buzz, data, monitor, offLed, onLed, otherLed, pot, pushButton, slideSwitch
- wire segments 199 -> 227

Commit message: Almost done
Parts:
- removed C2: C_Small, Capacitor_THT:C_Disc_D3.4mm_W2.1mm_P2.50mm, symbol Device:C_Small
- removed D6, D7, D8, D9: DIODE, Diode_THT:D_A-405_P2.54mm_Vertical_AnodeUp, symbol pspice:DIODE
- added C2: C, Capacitor_THT:C_Radial_D5.0mm_H11.0mm_P2.00mm, symbol Device:C
- added D1: D, Diode_THT:D_A-405_P7.62mm_Horizontal, symbol Device:D
- added Q4, Q5, Q6: BC547, Package_TO_SOT_THT:TO-92_Inline, symbol Transistor_BJT:BC547
- added R14: R, Resistor_THT:R_Axial_DIN0207_L6.3mm_D2.5mm_P10.16mm_Horizontal, symbol Device:R
- added R15, R16, R17: R, Resistor_THT:R_Axial_DIN0204_L3.6mm_D1.6mm_P2.54mm_Vertical, symbol Device:R
- D4, D5: footprint Diode_THT:D_A-405_P2.54mm_Vertical_AnodeUp -> Diode_THT:D_A-405_P7.62mm_Horizontal
Connections:
- wire segments 227 -> 221
Changed lines of the file:
@@
 F 0 "D4" V 10304 5028 50  0000 L CNN
 F 1 "DIODE" V 10395 5028 50  0000 L CNN
-F 2 "Diode_THT:D_A-405_P2.54mm_Vertical_AnodeUp" H 10350 4900 50  0001 C CNN
+F 2 "Diode_THT:D_A-405_P7.62mm_Horizontal" H 10350 4900 50  0001 C CNN
 F 3 "" H 10350 4900 50  0001 C CNN
 	1    10350 4900
@@
 F 0 "D5" V 10304 5928 50  0000 L CNN
 F 1 "DIODE" V 10395 5928 50  0000 L CNN
-F 2 "Diode_THT:D_A-405_P2.54mm_Vertical_AnodeUp" H 10350 5800 50  0001 C CNN
+F 2 "Diode_THT:D_A-405_P7.62mm_Horizontal" H 10350 5800 50  0001 C CNN
 F 3 "" H 10350 5800 50  0001 C CNN
 	1    10350 5800
@@
 L Connector:Screw_Terminal_01x02 J2
 U 1 1 5D944546
-P 9250 3300
-F 0 "J2" H 9170 2975 50  0000 C CNN
-F 1 "Screw_Terminal_01x02" H 9170 3066 50  0000 C CNN
-F 2 "TerminalBlock:TerminalBlock_bornier-2_P5.08mm" H 9250 3300 50  0001 C CNN
-F 3 "~" H 9250 3300 50  0001 C CNN
-	1    9250 3300
-	-1   0    0    1
-$EndComp
-Connection ~ 9450 3300
+P 9350 3200
+F 0 "J2" H 9270 2875 50  0000 C CNN
+F 1 "Screw_Terminal_01x02" H 9270 2966 50  0000 C CNN
+F 2 "TerminalBlock:TerminalBlock_bornier-2_P5.08mm" H 9350 3200 50  0001 C CNN
+F 3 "~" H 9350 3200 50  0001 C CNN
+	1    9350 3200
+	1    0    0    -1
+$EndComp
 $Comp
 L Connector:Screw_Terminal_01x02 J1
@@
 	6050 4300 8600 4300
 Wire Wire Line
-	5800 3400 9100 3400
-Wire Wire Line
 	8750 3900 9700 3900
 Wire Wire Line
 	10150 3050 11750 3050
-$Comp
-L pspice:DIODE D6
-U 1 1 5D9D48F2
-P 12500 4950
-F 0 "D6" H 12500 5215 50  0000 C CNN
-F 1 "DIODE" H 12500 5124 50  0000 C CNN
-F 2 "Diode_THT:D_A-405_P2.54mm_Vertical_AnodeUp" H 12500 4950 50  0001 C CNN
-F 3 "" H 12500 4950 50  0001 C CNN
-	1    12500 4950
-	1    0    0    -1
-$EndComp
-$Comp
-L pspice:DIODE D7
-U 1 1 5D9D4BD2
-P 12500 5500
-F 0 "D7" H 12500 5765 50  0000 C CNN
-F 1 "DIODE" H 12500 5674 50  0000 C CNN
-F 2 "Diode_THT:D_A-405_P2.54mm_Vertical_AnodeUp" H 12500 5500 50  0001 C CNN
-F 3 "" H 12500 5500 50  0001 C CNN
-	1    12500 5500
-	1    0    0    -1
-$EndComp
-$Comp
-L pspice:DIODE D8
-U 1 1 5D9D4C4C
-P 13250 4950
-F 0 "D8" H 13250 5215 50  0000 C CNN
-F 1 "DIODE" H 13250 5124 50  0000 C CNN
-F 2 "Diode_THT:D_A-405_P2.54mm_Vertical_AnodeUp" H 13250 4950 50  0001 C CNN
-F 3 "" H 13250 4950 50  0001 C CNN
-	1    13250 4950
-	1    0    0    -1
-$EndComp
-$Comp
-L pspice:DIODE D9
-U 1 1 5D9D4DE4
-P 13250 5500
-F 0 "D9" H 13250 5765 50  0000 C CNN
-F 1 "DIODE" H 13250 5674 50  0000 C CNN
-F 2 "Diode_THT:D_A-405_P2.54mm_Vertical_AnodeUp" H 13250 5500 50  0001 C CNN
-F 3 "" H 13250 5500 50  0001 C CNN
-	1    13250 5500
-	1    0    0    -1
-$EndComp
 $Comp
 L pspice:INDUCTOR L1
 U 1 1 5D9D4F0D
-P 12000 5200
-F 0 "L1" V 11954 5278 50  0000 L CNN
-F 1 "INDUCTOR" V 12045 5278 50  0000 L CNN
-F 2 "Inductor_THT:L_Axial_L9.5mm_D4.0mm_P12.70mm_Horizontal_Fastron_SMCC" H 12000 5200 50  0001 C CNN
-F 3 "" H 12000 5200 50  0001 C CNN
-	1    12000 5200
+P 13350 1200
+F 0 "L1" V 13304 1278 50  0000 L CNN
+F 1 "INDUCTOR" V 13395 1278 50  0000 L CNN
+F 2 "Inductor_THT:L_Axial_L9.5mm_D4.0mm_P12.70mm_Horizontal_Fastron_SMCC" H 13350 1200 50  0001 C CNN
+F 3 "" H 13350 1200 50  0001 C CNN
+	1    13350 1200
 	0    -1   -1   0
 $EndComp
-$Comp
-L Device:C_Small C2
-U 1 1 5D9D50DB
-P 13650 5200
-F 0 "C2" H 13742 5246 50  0000 L CNN
-F 1 "C_Small" H 13742 5155 50  0000 L CNN
-F 2 "Capacitor_THT:C_Disc_D3.4mm_W2.1mm_P2.50mm" H 13650 5200 50  0001 C CNN
-F 3 "~" H 13650 5200 50  0001 C CNN
-	1    13650 5200
-	1    0    0    -1
-$EndComp
-Wire Wire Line
-	12850 4950 13050 4950
-Wire Wire Line
-	13050 5500 12850 5500
-Wire Wire Line
-	12000 4950 12000 4600
-Wire Wire Line
-	12000 4600 12850 4600
-Wire Wire Line
-	12850 4600 12850 4950
-Connection ~ 12850 4950
-Wire Wire Line
-	12700 4950 12850 4950
-Wire Wire Line
-	12000 5450 12000 5800
-Wire Wire Line
-	12000 5800 12850 5800
-Wire Wire Line
-	12850 5800 12850 5500
-Connection ~ 12850 5500
-Wire Wire Line
-	12850 5500 12700 5500
-Wire Wire Line
-	12300 4950 12300 5500
-Wire Wire Line
-	12300 5500 12300 6000
-Wire Wire Line
-	12300 6000 12950 6000
-Wire Wire Line
-	13650 6000 13650 5300
-Connection ~ 12300 5500
-Wire Wire Line
-	13450 5500 13450 4950
-Wire Wire Line
-	13450 4950 13650 4950
-Connection ~ 13450 4950
-Wire Wire Line
-	13650 4950 13650 5100
-Wire Wire Line
-	12950 6000 12950 6700
-Wire Wire Line
-	12950 6700 11750 6700
-Wire Wire Line
-	12950 6000 13650 6000
-Connection ~ 12950 6000
-Connection ~ 11750 6700
-Wire Wire Line
-	13450 5500 13450 6300
-Wire Wire Line
-	13450 6300 9400 6300
-Connection ~ 13450 5500
-Wire Wire Line
-	9400 6300 9400 6050
-Wire Wire Line
-	9400 6050 6650 6050
-Wire Wire Line
-	6650 6050 6650 5950
 Wire Wire Line
 	9700 3200 9850 3200
@@
 	9700 3100 9700 3200
 Connection ~ 9700 3200
-Wire Wire Line
-	9450 3200 9550 3200
 Connection ~ 9550 3200
 Wire Wire Line
@@
 $EndComp
 Wire Wire Line
-	11750 3050 11750 4400
+	11750 3050 11750 3400
 Wire Wire Line
 	10900 4400 11750 4400
@@
 	1    0    0    -1
 $EndComp
-Wire Wire Line
-	7200 8750 8150 8750
 Wire Wire Line
 	7500 6300 7750 6300
@@
 buzz
 Wire Wire Line
+	7200 8750 8150 8750
+$Comp
+L Transistor_BJT:BC547 Q6
+U 1 1 5D9FED94
+P 13350 2000
+F 0 "Q6" V 13586 2000 50  0000 C CNN
+F 1 "BC547" V 13677 2000 50  0000 C CNN
+F 2 "Package_TO_SOT_THT:TO-92_Inline" H 13550 1925 50  0001 L CIN
+F 3 "http://www.fairchildsemi.com/ds/BC/BC547.pdf" H 13350 2000 50  0001 L CNN
+	1    13350 2000
+	0    1    1    0
+$EndComp
+$Comp
+L Transistor_BJT:BC547 Q5
+U 1 1 5D9FEEFB
+P 13000 2350
+F 0 "Q5" V 13236 2350 50  0000 C CNN
+F 1 "BC547" V 13327 2350 50  0000 C CNN
+F 2 "Package_TO_SOT_THT:TO-92_Inline" H 13200 2275 50  0001 L CIN
+F 3 "http://www.fairchildsemi.com/ds/BC/BC547.pdf" H 13000 2350 50  0001 L CNN
+	1    13000 2350
+	0    1    1    0
+$EndComp
+$Comp
+L Transistor_BJT:BC547 Q4
+U 1 1 5D9FEF99
+P 12600 2650
+F 0 "Q4" V 12836 2650 50  0000 C CNN
+F 1 "BC547" V 12927 2650 50  0000 C CNN
+F 2 "Package_TO_SOT_THT:TO-92_Inline" H 12800 2575 50  0001 L CIN
+F 3 "http://www.fairchildsemi.com/ds/BC/BC547.pdf" H 12600 2650 50  0001 L CNN
+	1    12600 2650
+	0    1    1    0
+$EndComp
+$Comp
+L Device:R R17
+U 1 1 5D9FF036
+P 13550 2250
+F 0 "R17" H 13620 2296 50  0000 L CNN
+F 1 "R" H 13620 2205 50  0000 L CNN
+F 2 "Resistor_THT:R_Axial_DIN0204_L3.6mm_D1.6mm_P2.54mm_Vertical" V 13480 2250 50  0001 C CNN
+F 3 "~" H 13550 2250 50  0001 C CNN
+	1    13550 2250
+	1    0    0    -1
+$EndComp
+$Comp
+L Device:R R16
+U 1 1 5D9FF104
+P 13200 2600
+F 0 "R16" H 13270 2646 50  0000 L CNN
+F 1 "R" H 13270 2555 50  0000 L CNN
+F 2 "Resistor_THT:R_Axial_DIN0204_L3.6mm_D1.6mm_P2.54mm_Vertical" V 13130 2600 50  0001 C CNN
+F 3 "~" H 13200 2600 50  0001 C CNN
+	1    13200 2600
+	1    0    0    -1
+$EndComp
+$Comp
+L Device:R R15
+U 1 1 5D9FF192
+P 12800 2900
+F 0 "R15" H 12870 2946 50  0000 L CNN
+F 1 "R" H 12870 2855 50  0000 L CNN
+F 2 "Resistor_THT:R_Axial_DIN0204_L3.6mm_D1.6mm_P2.54mm_Vertical" V 12730 2900 50  0001 C CNN
+F 3 "~" H 12800 2900 50  0001 C CNN
+	1    12800 2900
+	1    0    0    -1
+$EndComp
+$Comp
+L Device:D D1
+U 1 1 5DA0D55E
+P 12150 2950
+F 0 "D1" V 12196 2871 50  0000 R CNN
+F 1 "D" V 12105 2871 50  0000 R CNN
+F 2 "Diode_THT:D_A-405_P7.62mm_Horizontal" H 12150 2950 50  0001 C CNN
+F 3 "~" H 12150 2950 50  0001 C CNN
+	1    12150 2950
+	0    -1   -1   0
+$EndComp
+$Comp
+L Device:C C2
+U 1 1 5DA0D6B3
+P 11950 3250
+F 0 "C2" H 12065 3296 50  0000 L CNN
+F 1 "C" H 12065 3205 50  0000 L CNN
+F 2 "Capacitor_THT:C_Radial_D5.0mm_H11.0mm_P2.00mm" H 11988 3100 50  0001 C CNN
+F 3 "~" H 11950 3250 50  0001 C CNN
+	1    11950 3250
+	1    0    0    -1
+$EndComp
+$Comp
+L Device:R R14
+U 1 1 5DA0D756
+P 12150 3250
+F 0 "R14" H 12220 3296 50  0000 L CNN
+F 1 "R" H 12220 3205 50  0000 L CNN
+F 2 "Resistor_THT:R_Axial_DIN0207_L6.3mm_D2.5mm_P10.16mm_Horizontal" V 12080 3250 50  0001 C CNN
+F 3 "~" H 12150 3250 50  0001 C CNN
+	1    12150 3250
+	1    0    0    -1
+$EndComp
+Wire Wire Line
+	13350 1450 13350 1800
+Wire Wire Line
+	13150 2100 13000 2100
+Wire Wire Line
+	13000 2100 13000 2150
+Wire Wire Line
+	12800 2450 12600 2450
+Wire Wire Line
+	9850 3300 12800 3300
+Wire Wire Line
+	13550 3300 13550 2400
+Connection ~ 9850 3300
+Wire Wire Line
+	13200 2750 13200 3300
+Connection ~ 13200 3300
+Wire Wire Line
+	13200 3300 13550 3300
+Wire Wire Line
+	12800 3050 12800 3300
+Connection ~ 12800 3300
+Wire Wire Line
+	12800 3300 13200 3300
+Wire Wire Line
+	12400 2750 12150 2750
+Wire Wire Line
+	12150 2750 12150 2800
+Wire Wire Line
+	11950 3400 12150 3400
+Wire Wire Line
+	11950 3100 12150 3100
+Connection ~ 12150 3100
+Wire Wire Line
+	11950 3400 11750 3400
+Connection ~ 11950 3400
+Connection ~ 11750 3400
+Wire Wire Line
+	11750 3400 11750 4400
+Wire Wire Line
+	11950 3100 11150 3100
+Wire Wire Line
+	11150 3100 11150 2650
+Connection ~ 11950 3100
+Text Label 11150 2650 0    50   ~ 0
+monitor
+Wire Wire Line
+	5800 3400 9100 3400
+Wire Wire Line
+	9150 3200 9550 3200
+Wire Wire Line
+	9150 3300 9450 3300
+Wire Wire Line
+	7400 8150 8150 8150
+Wire Wire Line
+	7500 8050 8150 8050
+Wire Wire Line
+	7300 8250 8150 8250
+Wire Wire Line
+	7200 8350 8150 8350
+Wire Wire Line
+	7500 8450 8150 8450
+Wire Wire Line
+	7400 8550 8150 8550
+Wire Wire Line
 	7300 8650 8150 8650
-Wire Wire Line
-	7400 8550 8150 8550
-Wire Wire Line
-	7500 8450 8150 8450
-Wire Wire Line
-	7200 8350 8150 8350
-Wire Wire Line
-	7300 8250 8150 8250
-Wire Wire Line
-	7500 8050 8150 8050
-Wire Wire Line
-	7400 8150 8150 8150
 Wire Bus Line
 	10750 7950 10750 8950
@@
 Wire Bus Line
 	8000 7900 8000 8950
+Connection ~ 9450 3300
 $EndSCHEMATC

Commit message: PCB Layout  perfectly done
Parts:
- removed C1, C2: C, Capacitor_THT:C_Radial_D5.0mm_H11.0mm_P2.00mm, symbol Device:C
- removed L1: INDUCTOR, Inductor_THT:L_Axial_L9.5mm_D4.0mm_P12.70mm_Horizontal_Fastron_SMCC, symbol pspice:INDUCTOR
- added ANT1: ANT, Connector_Wire:SolderWirePad_1x01_Drill0.8mm, symbol connectors:HEADER-1x01
- added C1: 10uF, Capacitor_THT:CP_Radial_D4.0mm_P2.00mm, symbol Device:CP1
- added C2: 100uF, Capacitor_THT:CP_Radial_D4.0mm_P2.00mm, symbol Device:CP1
- R1, R10, R11, R2, R3, R4, R5, R6, R7, R8, R9: value R -> 220
- R12: value R -> 10K
- R13, R15: value R -> 1K
- R14: value R -> 2.2K
- R16: value R -> 100K
- R17: value R -> 1M
- R18: renamed from 10K2; value R -> 1K
- R19: renamed from 10K3; value R -> 1K
- R20: renamed from 1K1; value R -> 1K
- R21: renamed from 10K1; value R -> 10K
- renumbered digit2 to d2, digit2.1 to d2.1, digit3 to d3, digit3.1 to d3.1, green1 to g1, red1 to r1, yellow1 to y1
Connections:
- net labels added: offRelay, onRelay
