File: PCB Layout Files Kicad/Smartarter - 40/Smartarter.kicad_pcb (KiCad board)
At the start: 2 copper layers, 135.5 x 111.5 mm, 51 parts, among them J1 Screw_Terminal_01x02, J2 Screw_Terminal_01x02, K1 onRelay, K2 offRelay, Q1 BC547, Q2 BC547, Q3 BC547, SW1 SW_Push, U1 74164, U2 KCSA02-107, U3 slideSwitch, U4 7414, U5 KCSA02-107, U6 KCSA02-107, U7 KCSA02-107

Commit message: all tracks set in 40; double check the connections and HOLA ;)
Parts:
- removed the REF** at (75.2, 196.1)
- removed the REF** at (100.0, 196.1)
- removed U3: slideSwitch, Button_Switch_THT:SW_6-Pin-Switch_Self_Lock_DPDT_Latching
- added REF**: SolderWirePad_1x01_Drill2.5mm, Connector_Wire:SolderWirePad_1x01_Drill2.5mm, F.Cu at (99.7, 196.2)
- added SW2: SW_DPDT_x2, Button_Switch_THT:SW_6-Pin-Switch_Self_Lock_DPDT_Latching, B.Cu at (162.4, 162.0)
- added digit2: HEADER-1x01, Connector_Wire:SolderWirePad_1x01_Drill0.8mm, F.Cu at (67.0, 148.6)
- added digit2.1: HEADER-1x01, Connector_Wire:SolderWirePad_1x01_Drill0.8mm, F.Cu at (117.5, 148.6)
- added digit3: HEADER-1x01, Connector_Wire:SolderWirePad_1x01_Drill0.8mm, F.Cu at (80.4, 148.6)
- added digit3.1: HEADER-1x01, Connector_Wire:SolderWirePad_1x01_Drill0.8mm, F.Cu at (124.8, 148.6)
- L1: moved to B.Cu
- moved U7414 29.8 mm to (139.7, 128.1)
- moved C1 29.8 mm to (139.8, 134.1)
- moved L1 6.94 mm to (86.4, 196.3), turned to 180 degrees
- renumbered RV1 to POT1, U4 to U7414, U1 to U74164, D1 to green, D1 to green1, K2 to offRelay1, K1 to onRelay1, D2 to red, D2 to red1, D3 to yellow, D3 to yellow1
Connections:
- net Net-(A1-Pad14) renamed /monitor
- net Net-(A1-Pad18) renamed /pushButton
- net Net-(A1-Pad9) renamed /slideSwitch
- A1 pad 10: (no net) -> /pot
- A1 pad 11: (no net) -> /data
- A1 pad 12: (no net) -> /CLK
- A1 pad 13: (no net) -> /buzz
- A1 pad 15: (no net) -> /otherLed
- A1 pad 16: (no net) -> /offLed
- A1 pad 17: (no net) -> /onLed
- A1 pad 19: (no net) -> Net-(A1-Pad19)
- A1 pad 20: (no net) -> /D4
- A1 pad 21: (no net) -> Net-(A1-Pad21)
- A1 pad 22: (no net) -> /D1
- L1 pad 1: Net-(D6-Pad2) -> Net-(D7-Pad2)
- L1 pad 2: Net-(D7-Pad2) -> Net-(D6-Pad2)
- POT1 pad 2: (no net) -> /pot
- R1 pad 1: (no net) -> /onLed
- R1 pad 2: Net-(D1-Pad2) -> Net-(R1-Pad2)
- R13 pad 2: (no net) -> /buzz
- R2 pad 1: (no net) -> /offLed
- R2 pad 2: Net-(D2-Pad2) -> Net-(R2-Pad2)
- R3 pad 1: (no net) -> /otherLed
- R3 pad 2: Net-(D3-Pad2) -> Net-(R3-Pad2)
- U2 pad 3: (no net) -> /D1
- U5 pad 8: (no net) -> Net-(U5-Pad8)
- U6 pad 8: (no net) -> Net-(U6-Pad8)
- U7 pad 8: (no net) -> /D4
- U74164 pad 2: (no net) -> /data
- U74164 pad 8: (no net) -> /CLK
- green pad 2: Net-(D1-Pad2) -> (no net)
- green1 pad 2: Net-(D1-Pad2) -> Net-(R1-Pad2)
- red pad 2: Net-(D2-Pad2) -> (no net)
- red1 pad 2: Net-(D2-Pad2) -> Net-(R2-Pad2)
- yellow pad 2: Net-(D3-Pad2) -> (no net)
- yellow1 pad 2: Net-(D3-Pad2) -> Net-(R3-Pad2)
Routing:
- net (no net): track 450.8 -> 199.8 mm
- net GND: track 556.1 -> 431.7 mm
- net /D1: track 0.00 -> 87.6 mm
- net /pot: track 0.00 -> 86.1 mm
- net /data: track 0.00 -> 60.8 mm
- net /onLed: track 0.00 -> 50.7 mm
- net /CLK: track 0.00 -> 39.3 mm
- net /D4: track 0.00 -> 36.7 mm
- net /offLed: track 0.00 -> 35.7 mm
- net /pushButton: track 64.7 -> 31.7 mm
- net Net-(1K1-Pad2): track 79.3 -> 47.8 mm
- net Net-(D6-Pad2): track 165.9 -> 144.1 mm
- net /otherLed: track 0.00 -> 20.9 mm
- net /buzz: track 0.00 -> 19.0 mm
- net /A0: track 56.6 -> 74.4 mm
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Other:
- board size 135.5 x 111.5 mm -> 135.5 x 112.3 mm
- board text added: "+"
- board text added: "-"
- board text added: "12V"
- board text added: "5V"
- board text added: "BZ"
- board text added: "GND"

Commit message: Almost done
Parts:
- removed D6, D7, D8, D9: DIODE, Diode_THT:D_A-405_P2.54mm_Vertical_AnodeUp
- removed REF**: SolderWirePad_1x01_Drill2.5mm, Connector_Wire:SolderWirePad_1x01_Drill2.5mm
- removed green: onLED, LED_THT:LED_Rectangular_W3.9mm_H1.8mm
- removed red: offLED, LED_THT:LED_Rectangular_W3.9mm_H1.8mm
- removed the red1 at (77.1, 143.2)
- removed yellow: otherLED, LED_THT:LED_Rectangular_W3.9mm_H1.8mm
- added D1: D, Diode_THT:D_A-405_P7.62mm_Horizontal, F.Cu at (138.3, 104.7)
- added Q4: BC547, Package_TO_SOT_THT:TO-92_Inline, F.Cu at (156.4, 116.8)
- added Q5: BC547, Package_TO_SOT_THT:TO-92_Inline, F.Cu at (158.7, 107.2)
- added Q6: BC547, Package_TO_SOT_THT:TO-92_Inline, F.Cu at (143.9, 113.9)
- added R14: R, Resistor_THT:R_Axial_DIN0207_L6.3mm_D2.5mm_P10.16mm_Horizontal, F.Cu at (109.9, 98.5)
- added R15: R, Resistor_THT:R_Axial_DIN0204_L3.6mm_D1.6mm_P2.54mm_Vertical, F.Cu at (156.3, 124.1)
- added R16: R, Resistor_THT:R_Axial_DIN0204_L3.6mm_D1.6mm_P2.54mm_Vertical, F.Cu at (162.7, 116.9)
- added R17: R, Resistor_THT:R_Axial_DIN0204_L3.6mm_D1.6mm_P2.54mm_Vertical, F.Cu at (143.9, 118.5)
- added green1: onLED, LED_THT:LED_Rectangular_W3.9mm_H1.8mm, F.Cu at (59.3, 143.0)
- added red1: offLED, LED_THT:LED_Rectangular_W3.9mm_H1.8mm, F.Cu at (69.7, 143.0)
- added red1: offLED, LED_THT:LED_Rectangular_W3.9mm_H1.8mm, F.Cu at (77.4, 143.0)
- added yellow1: otherLED, LED_THT:LED_Rectangular_W3.9mm_H1.8mm, F.Cu at (87.9, 143.0)
- C2: value C_Small -> C; footprint Capacitor_THT:C_Disc_D3.4mm_W2.1mm_P2.50mm -> Capacitor_THT:C_Radial_D5.0mm_H11.0mm_P2.00mm
- D4, D5: footprint Diode_THT:D_A-405_P2.54mm_Vertical_AnodeUp -> Diode_THT:D_A-405_P7.62mm_Horizontal; moved to F.Cu
- L1: moved to F.Cu
- moved L1 193.9 mm to (150.0, 13.1), turned to 0 degrees
- moved J2 105.4 mm to (70.3, 197.6), turned to 0 degrees
- moved J1 105.4 mm to (59.2, 197.5), turned to 0 degrees
- moved Q3 86.9 mm to (46.5, 184.3), turned to 0 degrees
- moved C2 55.0 mm to (116.4, 102.8)
- moved 10K3 36.6 mm to (58.5, 186.9)
- moved Q1 35.6 mm to (53.6, 192.1)
- moved Q2 32.9 mm to (46.5, 190.0)
- moved R13 27.1 mm to (61.9, 107.5)
- moved D5 25.1 mm to (74.7, 181.7), turned to 270 degrees
- moved offRelay1 24.8 mm to (82.5, 176.1)
- moved onRelay1 24.8 mm to (115.2, 176.1)
- moved 10K2 24.5 mm to (54.0, 182.9)
- moved D4 21.7 mm to (79.9, 181.7), turned to 270 degrees
- moved yellow1 7.15 mm to (80.1, 143.0), turned to 0 degrees
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Connections:
- J2 pad 1: +5V -> GND
- J2 pad 2: GND -> +5V
- L1 pad 2: Net-(D6-Pad2) -> (no net)
Routing:
- net Net-(L1-Pad1): track 168.6 -> 0.00 mm
- net Net-(D6-Pad2): track 144.1 -> 0.00 mm
- net +12V: track 167.3 -> 23.8 mm
- net +5V: track 230.2 -> 355.0 mm
- net Net-(Q3-Pad2): track 7.75 -> 84.3 mm
- net GND: track 431.7 -> 370.5 mm
- net /buzz: track 19.0 -> 47.8 mm
- net /monitor: track 56.1 -> 36.8 mm
- net Net-(D1-Pad2): track 0.00 -> 15.4 mm
- net Net-(J1-Pad2): track 10.8 -> 25.7 mm
- net Net-(Q5-Pad2): track 0.00 -> 14.5 mm
- net Net-(Q5-Pad1): track 0.00 -> 12.8 mm
- net (no net): track 199.8 -> 210.7 mm
- net Net-(1K1-Pad2): track 47.8 -> 57.8 mm
- net Net-(Q4-Pad2): track 0.00 -> 9.27 mm
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Other:
- outline, holes or cut-outs redrawn

Commit message: PCB Layout  perfectly done
Parts:
- removed 10K2, 10K3: R, Resistor_THT:R_Axial_DIN0207_L6.3mm_D2.5mm_P10.16mm_Horizontal
- removed L1: INDUCTOR, Inductor_THT:L_Axial_L9.5mm_D4.0mm_P12.70mm_Horizontal_Fastron_SMCC
- added ANT1: ANT, Connector_Wire:SolderWirePad_1x01_Drill0.8mm, F.Cu at (150.2, 20.4)
- added R18: 1K, Resistor_THT:R_Axial_DIN0207_L6.3mm_D2.5mm_P10.16mm_Horizontal, F.Cu at (51.6, 106.6)
- added R19: 1K, Resistor_THT:R_Axial_DIN0207_L6.3mm_D2.5mm_P10.16mm_Horizontal, F.Cu at (56.2, 110.8)
- C1: value C -> 10uF; footprint Capacitor_THT:C_Radial_D5.0mm_H11.0mm_P2.00mm -> Capacitor_THT:CP_Radial_D4.0mm_P2.00mm
- C2: value C -> 100uF; footprint Capacitor_THT:C_Radial_D5.0mm_H11.0mm_P2.00mm -> Capacitor_THT:CP_Radial_D4.0mm_P2.00mm
- R1, R10, R11, R2, R3, R4, R5, R6, R7, R8, R9: value R -> 220
- R12: value R -> 10K
- R13, R15: value R -> 1K
- R14: value R -> 2.2K
- R16: value R -> 100K
- R17: value R -> 1M
- R20: renamed from 1K1; value R -> 1K
- R21: renamed from 10K1; value R -> 10K
- moved J2 76.1 mm to (67.9, 121.5)
- moved POT1 76.1 mm to (110.7, 93.8)
- moved Q3 76.1 mm to (44.1, 108.2)
- moved Q6 76.1 mm to (141.5, 37.8)
- moved R11 76.1 mm to (94.9, 48.3)
- moved R16 76.1 mm to (160.3, 40.8)
- moved R20 76.1 mm to (128.3, 79.7)
- moved R4 76.1 mm to (48.4, 72.8)
- moved R5 76.1 mm to (53.1, 72.8)
- moved R8 76.1 mm to (59.5, 95.3)
- moved SW1 76.1 mm to (134.4, 81.3)
- moved U74164 76.1 mm to (68.2, 45.0)
- moved g1 76.1 mm to (56.9, 66.9)
- moved g1 76.1 mm to (64.7, 66.9)
- moved offRelay1 76.1 mm to (80.0, 100.0)
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- renumbered digit2 to d2, digit2.1 to d2.1, digit3 to d3, digit3.1 to d3.1, green1 to g1, red1 to r1, yellow1 to y1
Connections:
- A1 pad 1: (no net) -> Net-(A1-Pad1)
- A1 pad 2: (no net) -> Net-(A1-Pad2)
- A1 pad 23: (no net) -> Net-(A1-Pad23)
- A1 pad 24: (no net) -> Net-(A1-Pad24)
- A1 pad 25: (no net) -> Net-(A1-Pad25)
- A1 pad 26: (no net) -> /offRelay
- A1 pad 27: (no net) -> /onRelay
- A1 pad 28: (no net) -> Net-(A1-Pad28)
- A1 pad 29: (no net) -> Net-(A1-Pad29)
- A1 pad 3: (no net) -> Net-(A1-Pad3)
- A1 pad 30: (no net) -> Net-(A1-Pad30)
- A1 pad 31: (no net) -> Net-(A1-Pad31)
- A1 pad 32: (no net) -> Net-(A1-Pad32)
- A1 pad 4: (no net) -> Net-(A1-Pad4)
- A1 pad 5: (no net) -> Net-(A1-Pad5)
- A1 pad 7: (no net) -> Net-(A1-Pad7)
- U2 pad 8: (no net) -> Net-(U2-Pad8)
- U5 pad 3: (no net) -> Net-(U5-Pad3)
- U6 pad 3: (no net) -> Net-(U6-Pad3)
- U7 pad 3: (no net) -> Net-(U7-Pad3)
- offRelay1 pad 2: (no net) -> Net-(offRelay1-Pad2)
- offRelay1 pad 3: (no net) -> Net-(offRelay1-Pad3)
- offRelay1 pad 4: (no net) -> Net-(offRelay1-Pad4)
- onRelay1 pad 2: (no net) -> Net-(onRelay1-Pad2)
- onRelay1 pad 3: (no net) -> Net-(onRelay1-Pad3)
- onRelay1 pad 4: (no net) -> Net-(onRelay1-Pad4)
Routing:
- net (no net): track 210.7 -> 0.00 mm
- net /onRelay: track 0.00 -> 105.0 mm
- net /offRelay: track 0.00 -> 103.5 mm
- net Net-(ANT1-Pad1): track 0.00 -> 20.5 mm
- net GND: track 370.5 -> 367.0 mm
- net /A5: track 72.7 -> 70.9 mm
- net +5V: track 355.0 -> 353.3 mm
- net /A4: track 63.8 -> 62.3 mm
- net /A0: track 74.4 -> 73.4 mm
- net Net-(R8-Pad2): track 106.1 -> 107.1 mm
- net /D1: track 87.6 -> 88.1 mm
Other:
- board size 135.5 x 112.3 mm -> 131.1 x 112.3 mm
- board text added: "A0"
- board text added: "A5"
- board text added: "Vin"
- board text added: "d1"
- board text added: "d4"
- board text removed: "+"
- board text removed: "-"
- board text removed: "12V 1A"
- board text removed: "5V 2A"
