File: PCB Layout Files Kicad/Smartarter-compact/Smartarter.sch (KiCad schematic (older format))
At the start: 50 parts, among them J1 Screw_Terminal_01x02, J2 Screw_Terminal_01x02, Q1 BC547, Q2 BC547, Q3 BC547, Q4 BC547, Q5 BC547, Q6 BC547, SW1 SW_Push, SW2 SW_DIP_x02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

Commit message: Ready for Ahmedabad
Parts:
- Q1, Q2, Q3, Q4, Q5, Q6: footprint Package_TO_SOT_THT:TO-92_Inline -> Package_TO_SOT_THT:TO-92_Inline_Wide
Changed lines of the file:
@@
 F 0 "Q1" H 9941 4946 50  0000 L CNN
 F 1 "BC547" H 9941 4855 50  0000 L CNN
-F 2 "Package_TO_SOT_THT:TO-92_Inline" H 9950 4825 50  0001 L CIN
+F 2 "Package_TO_SOT_THT:TO-92_Inline_Wide" H 9950 4825 50  0001 L CIN
 F 3 "http://www.fairchildsemi.com/ds/BC/BC547.pdf" H 9750 4900 50  0001 L CNN
 	1    9750 4900
@@
 F 0 "Q2" H 9941 5846 50  0000 L CNN
 F 1 "BC547" H 9941 5755 50  0000 L CNN
-F 2 "Package_TO_SOT_THT:TO-92_Inline" H 9950 5725 50  0001 L CIN
+F 2 "Package_TO_SOT_THT:TO-92_Inline_Wide" H 9950 5725 50  0001 L CIN
 F 3 "http://www.fairchildsemi.com/ds/BC/BC547.pdf" H 9750 5800 50  0001 L CNN
 	1    9750 5800
@@
 F 0 "Q3" H 5891 3246 50  0000 L CNN
 F 1 "BC547" H 5891 3155 50  0000 L CNN
-F 2 "Package_TO_SOT_THT:TO-92_Inline" H 5900 3125 50  0001 L CIN
+F 2 "Package_TO_SOT_THT:TO-92_Inline_Wide" H 5900 3125 50  0001 L CIN
 F 3 "http://www.fairchildsemi.com/ds/BC/BC547.pdf" H 5700 3200 50  0001 L CNN
 	1    5700 3200
@@
 F 0 "Q6" V 13586 2000 50  0000 C CNN
 F 1 "BC547" V 13677 2000 50  0000 C CNN
-F 2 "Package_TO_SOT_THT:TO-92_Inline" H 13550 1925 50  0001 L CIN
+F 2 "Package_TO_SOT_THT:TO-92_Inline_Wide" H 13550 1925 50  0001 L CIN
 F 3 "http://www.fairchildsemi.com/ds/BC/BC547.pdf" H 13350 2000 50  0001 L CNN
 	1    13350 2000
@@
 F 0 "Q5" V 13236 2350 50  0000 C CNN
 F 1 "BC547" V 13327 2350 50  0000 C CNN
-F 2 "Package_TO_SOT_THT:TO-92_Inline" H 13200 2275 50  0001 L CIN
+F 2 "Package_TO_SOT_THT:TO-92_Inline_Wide" H 13200 2275 50  0001 L CIN
 F 3 "http://www.fairchildsemi.com/ds/BC/BC547.pdf" H 13000 2350 50  0001 L CNN
 	1    13000 2350
@@
 F 0 "Q4" V 12836 2650 50  0000 C CNN
 F 1 "BC547" V 12927 2650 50  0000 C CNN
-F 2 "Package_TO_SOT_THT:TO-92_Inline" H 12800 2575 50  0001 L CIN
+F 2 "Package_TO_SOT_THT:TO-92_Inline_Wide" H 12800 2575 50  0001 L CIN
 F 3 "http://www.fairchildsemi.com/ds/BC/BC547.pdf" H 12600 2650 50  0001 L CNN
 	1    12600 2650
