File: PCB Layout Files Kicad/Smartarter-compact/Smartarter.kicad_pcb (KiCad board)
At the start: 2 copper layers, 101.6 x 76.2 mm, 50 parts, among them J1 Screw_Terminal_01x02, J2 Screw_Terminal_01x02, Q1 BC547, Q2 BC547, Q3 BC547, Q4 BC547, Q5 BC547, Q6 BC547, SW1 SW_Push, SW2 SW_DIP_x02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

Commit message: Ready for Ahmedabad
Parts:
- Q1, Q2, Q3, Q4, Q5, Q6: footprint Package_TO_SOT_THT:TO-92_Inline -> Package_TO_SOT_THT:TO-92_Inline_Wide
- moved R19 3.00 mm to (116.5, 129.2), turned to 180 degrees
- moved Q5 2.46 mm to (76.0, 106.9)
- moved R16 1.97 mm to (74.5, 112.0)
- moved Q4 1.97 mm to (64.6, 102.5)
- moved Q3 0.81 mm to (95.7, 127.9)
- moved R20 0.70 mm to (126.6, 70.2)
Routing:
- net GND: track 281.2 -> 326.8 mm
- net /D3: track 77.4 -> 101.6 mm
- net /pushButton: track 26.1 -> 46.0 mm
- net Net-(R5-Pad1): track 57.1 -> 70.7 mm
- net /monitor: track 95.2 -> 108.7 mm
- net Net-(C1-Pad1): track 73.1 -> 86.4 mm
- net Net-(R2-Pad1): track 40.7 -> 50.9 mm
- net Net-(R3-Pad1): track 38.3 -> 47.0 mm
- net /bz: track 15.3 -> 20.8 mm
- net /onRelay: track 49.7 -> 46.7 mm
- net +5V: track 289.6 -> 287.2 mm
- net Net-(Q2-Pad2): track 7.04 -> 5.81 mm
- net Net-(Q4-Pad2): track 5.89 -> 7.09 mm
- net Net-(R4-Pad2): track 5.97 -> 4.81 mm
- net Net-(D4-Pad2): track 24.3 -> 25.1 mm
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
Commit message: Finalized compact pcb layout
Parts:
- A1: value Arduino_Nano_v3.x -> Arduino_Nano
- POT1: value R_POT -> 10K
- Q1, Q2, Q3, Q4, Q5, Q6: value BC547 -> 547
- U1: value CA56-12EWA -> 4_Digit_7_Seg
- moved g1 0.82 mm to (75.4, 68.0)
- moved y1 0.80 mm to (102.1, 68.0)
- moved r1 0.40 mm to (85.3, 68.0)
- moved r2 0.40 mm to (92.2, 68.0)
Routing:
- net Net-(R2-Pad1): track 50.9 -> 53.0 mm
- net Net-(R1-Pad1): track 45.8 -> 45.0 mm
- net Net-(R3-Pad1): track 47.0 -> 46.2 mm
- net GND: track 326.8 -> 327.3 mm

Commit message: online backup, pcb display code and TODO some changes to be done in PCB
Other:
- board text added: "0"
- board text added: "1"
- board text added: "10"
- board text added: "11"
- board text added: "12"
- board text added: "2"
- board text added: "3"
- board text added: "4"
- board text added: "5"
- board text added: "6"
- board text added: "7"
- board text added: "8"
- board text added: "9"
- board text added: "A7"
- board text added: "D13"
- board text added: "D2"
- board text added: "D3"
Changed lines of the file:
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@@
   (general
     (thickness 1.6)
-    (drawings 10)
+    (drawings 32)
     (tracks 375)
     (zones 0)
@@
   )
   (setup
-    (last_trace_width 0.5)
+    (last_trace_width 0.25)
     (user_trace_width 0.5)
     (user_trace_width 1)
@@
     )
   )
+  (gr_text D13 (at 158.9 99.3) (layer F.SilkS)
+    (effects (font (size 1 1) (thickness 0.25)))
+  )
+  (gr_text 0 (at 151.4 99.2) (layer F.SilkS)
+    (effects (font (size 1 1) (thickness 0.25)))
+  )
+  (gr_text 1 (at 148.9 99.1) (layer F.SilkS)
+    (effects (font (size 1 1) (thickness 0.25)))
+  )
+  (gr_text 2 (at 146.3 99.3) (layer F.SilkS)
+    (effects (font (size 1 1) (thickness 0.25)))
+  )
+  (gr_text 3 (at 143.5 99.1) (layer F.SilkS)
+    (effects (font (size 1 1) (thickness 0.25)))
+  )
+  (gr_text 4 (at 141.1 99.1) (layer F.SilkS)
+    (effects (font (size 1 1) (thickness 0.25)))
+  )
+  (gr_text 5 (at 138.5 99.3) (layer F.SilkS)
+    (effects (font (size 1 1) (thickness 0.25)))
+  )
+  (gr_text 6 (at 136.2 99.2) (layer F.SilkS)
+    (effects (font (size 1 1) (thickness 0.25)))
+  )
+  (gr_text A7 (at 133.5 99.1) (layer F.SilkS)
+    (effects (font (size 1 1) (thickness 0.25)))
+  )
+  (gr_text 5V (at 130.8 99.1) (layer F.SilkS)
+    (effects (font (size 1 1) (thickness 0.25)))
+  )
+  (gr_text GND (at 131 111.1) (layer F.SilkS)
+    (effects (font (size 1 1) (thickness 0.25)))
+  )
+  (gr_text 12 (at 158.9 110.9) (layer F.SilkS)
+    (effects (font (size 1 1) (thickness 0.25)))
+  )
+  (gr_text 11 (at 156.4 111) (layer F.SilkS)
+    (effects (font (size 1 1) (thickness 0.25)))
+  )
+  (gr_text 10 (at 153.7 110.9) (layer F.SilkS)
+    (effects (font (size 1 1) (thickness 0.25)))
+  )
+  (gr_text 9 (at 151.3 110.9) (layer F.SilkS)
+    (effects (font (size 1 1) (thickness 0.25)))
+  )
+  (gr_text 8 (at 148.8 110.8) (layer F.SilkS)
+    (effects (font (size 1 1) (thickness 0.25)))
+  )
+  (gr_text 7 (at 146.1 111) (layer F.SilkS)
+    (effects (font (size 1 1) (thickness 0.25)))
+  )
+  (gr_text 6 (at 143.7 111) (layer F.SilkS)
+    (effects (font (size 1 1) (thickness 0.25)))
+  )
+  (gr_text 5 (at 140.9 110.8) (layer F.SilkS)
+    (effects (font (size 1 1) (thickness 0.25)))
+  )
+  (gr_text "4\n" (at 138.4 110.8) (layer F.SilkS)
+    (effects (font (size 1 1) (thickness 0.25)))
+  )
+  (gr_text D2 (at 133.5 111) (layer F.SilkS)
+    (effects (font (size 1 1) (thickness 0.25)))
+  )
+  (gr_text D3 (at 136.1 110.7) (layer F.SilkS)
+    (effects (font (size 1 1) (thickness 0.25)))
+  )
   (gr_arc (start 83.4 103.2) (end 83.4 102.4) (angle -180) (layer F.SilkS) (width 0.6))
